File: KiCad/Système_PCB/Système_PCB.kicad_sch (KiCad schematic)
At the start: 7 parts

Commit message: --Update PCB
Parts:
- removed R?: (no value), symbol Device:R
- removed R?: R, symbol Device:R
- added A1: (no value), symbol MCU_Module:Arduino_UNO_R3
- added R1: R, FootprintGamelGe2_v6:R_Axial_DIN0207_L6.3mm_D2.5mm_P10.16mm_Horizontal, symbol SymbGamelGe2_v6:R
- added R2: (no value), symbol SymbGamelGe2_v6:R
- D1: renamed from D?; value (none) -> 1N4001; footprint (none) -> Diode_THT:D_DO-41_SOD81_P10.16mm_Horizontal
- J1: renamed from J?; value (none) -> Autocom4; footprint (none) -> FootprintGamelGe2_v6:Autocom4
- J2: renamed from J?; value (none) -> Omnimate2; footprint (none) -> FootprintGamelGe2_v6:OmnimateSL-5,08_1x02_P5.08mm_Vertical
- gave numbers to parts that had none: 2
Connections:
- net GND: now also A1.29 (GND), R2.2
- net D1: now reaches Q1.1 (G)
- net D1: now also A1.16 (D1/TX), R2.1
- net Data_Out renamed D13
- net D13: now also A1.28 (D13), R1.1
- net VCC_Sensor renamed 5V
- net 5V: now also A1.5 (+5V), R1.2

Commit message: Change PCB
Parts:
- added C1: (no value), symbol SymbGamelGe2_v6:C
- added C2: Cp, FootprintGamelGe2_v6:CP_Radial_D10.0mm_P5.00mm, symbol SymbGamelGe2_v6:Cp
- added C?: C, FootprintGamelGe2_v6:C_Rect_L7.0mm_W2.5mm_P5.00mm, symbol SymbGamelGe2_v6:C
- A1: value (none) -> Arduino_UNO_R3; footprint (none) -> Module:Arduino_UNO_R3
- J3: value Omnimate2 -> (none); footprint FootprintGamelGe2_v6:OmnimateSL-5,08_1x02_P5.08mm_Vertical -> (none)
- Q1: value (none) -> IRL510; footprint (none) -> FootprintGamelGe2_v6:TO-220-3_Horizontal_TabDown
- R2: value (none) -> R; footprint (none) -> FootprintGamelGe2_v6:R_Axial_DIN0207_L6.3mm_D2.5mm_P10.16mm_Horizontal
Connections:
- net +12V: now also C2.1, C?.1
- net 5V: now also C1.1
- net GND: now also A1.6 (GND), A1.7 (GND), C1.2, C2.2, C?.2
- net A0: now reaches A1.9 (A0)
- net A0: now also J1.2 (Pin_2), R1.1
- removed net D13: A1.28 (D13), J1.2 (Pin_2), R1.1

Commit message: minor change
Parts:
- C1: value (none) -> C; footprint (none) -> FootprintGamelGe2_v6:C_Rect_L7.0mm_W2.5mm_P5.00mm
- J3: value (none) -> Omnimate2; footprint (none) -> FootprintGamelGe2_v6:OmnimateSL-5,08_1x02_P5.08mm_Vertical
- gave numbers to parts that had none: 1
Changed lines of the file:
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@@
       (effects (font (size 1.27 1.27)) (justify left))
     )
-    (property "Value" "" (id 1) (at 163.83 126.9999 0)
-      (effects (font (size 1.27 1.27)) (justify left))
-    )
-    (property "Footprint" "" (id 2) (at 160.9852 129.54 0)
+    (property "Value" "C" (id 1) (at 163.83 126.9999 0)
+      (effects (font (size 1.27 1.27)) (justify left))
+    )
+    (property "Footprint" "FootprintGamelGe2_v6:C_Rect_L7.0mm_W2.5mm_P5.00mm" (id 2) (at 160.9852 129.54 0)
       (effects (font (size 1.27 1.27)) hide)
     )
@@
       (effects (font (size 1.27 1.27)) (justify right))
     )
-    (property "Value" "" (id 1) (at 142.24 82.6776 0)
-      (effects (font (size 1.27 1.27)) (justify right))
-    )
-    (property "Footprint" "" (id 2) (at 146.05 81.28 0)
+    (property "Value" "Omnimate2" (id 1) (at 142.24 82.6776 0)
+      (effects (font (size 1.27 1.27)) (justify right))
+    )
+    (property "Footprint" "FootprintGamelGe2_v6:OmnimateSL-5,08_1x02_P5.08mm_Vertical" (id 2) (at 146.05 81.28 0)
       (effects (font (size 1.27 1.27)) hide)
     )
@@
   (symbol (lib_id "SymbGamelGe2_v6:C") (at 171.45 82.55 0) (unit 1)
     (in_bom yes) (on_board yes) (fields_autoplaced)
-    (property "Reference" "C?" (id 0) (at 175.26 81.2799 0)
+    (property "Reference" "C3" (id 0) (at 175.26 81.2799 0)
       (effects (font (size 1.27 1.27)) (justify left))
     )
@@
     )
     (path "/dfa79366-7445-4f78-8c0b-12e88ad4068f"
-      (reference "C?") (unit 1) (value "C") (footprint "FootprintGamelGe2_v6:C_Rect_L7.0mm_W2.5mm_P5.00mm")
+      (reference "C3") (unit 1) (value "C") (footprint "FootprintGamelGe2_v6:C_Rect_L7.0mm_W2.5mm_P5.00mm")
     )
     (path "/02d56d2c-b6b5-4ca1-9051-cd7f181a6d0c"
