File: KiCad/Système_PCB/Système_PCB.kicad_sch (KiCad schematic)
At the start: 11 parts, among them J1 Autocom4, J2 Omnimate2, J3 Omnimate2, Q1 IRL510

Commit message: -add PWM
Parts:
- C1, C3: value (none) -> 20n; footprint (none) -> FootprintGamelGe2_v6:C_Rect_L7.0mm_W2.5mm_P5.00mm
- C2: value (none) -> 100µ; footprint (none) -> FootprintGamelGe2_v6:CP_Radial_D5.0mm_P2.50mm
- Q1: value IRL510 -> (none); footprint FootprintGamelGe2_v6:TO-220-3_Horizontal_TabDown -> (none)
- R2: value (none) -> 4.7k; footprint (none) -> FootprintGamelGe2_v6:R_Axial_DIN0207_L6.3mm_D2.5mm_P10.16mm_Horizontal
Connections:
- net GND: now also Q1.3 (S); no longer Q1.2 (D)
- net at D1.2 (A), J2.1 (Pin_1): now also Q1.2 (D); no longer Q1.3 (S)
Other:
- moved on the sheet: Q1
Changed lines of the file:
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@@
   (junction (at 160.02 121.92) (diameter 0) (color 0 0 0 0)
-  )
-  (junction (at 199.39 99.06) (diameter 0) (color 0 0 0 0)
   )
   (junction (at 208.28 104.14) (diameter 0) (color 0 0 0 0)
@@
       (effects (font (size 1.27 1.27)) (justify left))
     )
-    (property "Value" "" (id 1) (at 165.1 83.1849 0)
-      (effects (font (size 1.27 1.27)) (justify left))
-    )
-    (property "Footprint" "" (id 2) (at 161.29 82.55 0)
+    (property "Value" "100µ" (id 1) (at 165.1 83.1849 0)
+      (effects (font (size 1.27 1.27)) (justify left))
+    )
+    (property "Footprint" "FootprintGamelGe2_v6:CP_Radial_D5.0mm_P2.50mm" (id 2) (at 161.29 82.55 0)
       (effects (font (size 1.27 1.27)) hide)
     )
@@
       (effects (font (size 1.27 1.27)) (justify left))
     )
-    (property "Value" "" (id 1) (at 163.83 126.9999 0)
-      (effects (font (size 1.27 1.27)) (justify left))
-    )
-    (property "Footprint" "" (id 2) (at 160.9852 129.54 0)
+    (property "Value" "20n" (id 1) (at 163.83 126.9999 0)
+      (effects (font (size 1.27 1.27)) (justify left))
+    )
+    (property "Footprint" "FootprintGamelGe2_v6:C_Rect_L7.0mm_W2.5mm_P5.00mm" (id 2) (at 160.9852 129.54 0)
       (effects (font (size 1.27 1.27)) hide)
     )
@@
       (effects (font (size 1.27 1.27)) (justify left))
     )
-    (property "Value" "" (id 1) (at 210.82 115.5699 0)
-      (effects (font (size 1.27 1.27)) (justify left))
-    )
-    (property "Footprint" "" (id 2) (at 206.502 114.3 90)
+    (property "Value" "4.7k" (id 1) (at 210.82 115.5699 0)
+      (effects (font (size 1.27 1.27)) (justify left))
+    )
+    (property "Footprint" "FootprintGamelGe2_v6:R_Axial_DIN0207_L6.3mm_D2.5mm_P10.16mm_Horizontal" (id 2) (at 206.502 114.3 90)
       (effects (font (size 1.27 1.27)) hide)
     )
@@
       (effects (font (size 1.27 1.27)) (justify left))
     )
-    (property "Value" "" (id 1) (at 175.26 83.8199 0)
-      (effects (font (size 1.27 1.27)) (justify left))
-    )
-    (property "Footprint" "" (id 2) (at 172.4152 86.36 0)
+    (property "Value" "20n" (id 1) (at 175.26 83.8199 0)
+      (effects (font (size 1.27 1.27)) (justify left))
+    )
+    (property "Footprint" "FootprintGamelGe2_v6:C_Rect_L7.0mm_W2.5mm_P5.00mm" (id 2) (at 172.4152 86.36 0)
       (effects (font (size 1.27 1.27)) hide)
     )
@@
     (pin "1")
   )
-  (symbol (lib_id "SymbGamelGe2_v6:IRL510") (at 201.93 104.14 180) (unit 1)
+  (symbol (lib_id "SymbGamelGe2_v6:IRL510") (at 201.93 104.14 0) (mirror y) (unit 1)
     (in_bom yes) (on_board yes) (fields_autoplaced)
     (property "Reference" "Q1" (id 0) (at 195.58 102.8699 0)
       (effects (font (size 1.27 1.27)) (justify left))
     )
-    (property "Value" "IRL510" (id 1) (at 195.58 105.4099 0)
-      (effects (font (size 1.27 1.27)) (justify left))
-    )
-    (property "Footprint" "FootprintGamelGe2_v6:TO-220-3_Horizontal_TabDown" (id 2) (at 195.58 102.235 0)
+    (property "Value" "" (id 1) (at 195.58 105.4099 0)
+      (effects (font (size 1.27 1.27)) (justify left))
+    )
+    (property "Footprint" "" (id 2) (at 195.58 106.045 0)
       (effects (font (size 1.27 1.27) italic) (justify left) hide)
     )
