File: KiCad/Système_PCB/Système_PCB.kicad_pcb (KiCad board)
At the start: 2 copper layers, 8 parts, among them J1 Autocom4, J2 Omnimate2, J3 Omnimate2, Q1 IRL510

Commit message: Change PCB
Parts:
- added C1: C, FootprintGamelGe2_v6:C_Rect_L7.0mm_W2.5mm_P5.00mm, F.Cu at (246.4, 81.3)
- added C2: Cp, FootprintGamelGe2_v6:CP_Radial_D10.0mm_P5.00mm, F.Cu at (217.2, 91.6)
- moved J1 1.27 mm to (251.4, 78.7)
- moved A1 0.25 mm to (215.3, 102.6)
Connections:
- A1 pad 28: /D13 -> unconnected-(A1-Pad28)
- A1 pad 6: unconnected-(A1-Pad6) -> GND
- A1 pad 7: unconnected-(A1-Pad7) -> GND
- A1 pad 9: unconnected-(A1-Pad9) -> /A0
- J1 pad 2: /D13 -> /A0
- R1 pad 1: /D13 -> /A0
Routing:
- net GND: track 50.0 -> 154.9 mm, vias 0 -> 2
- net /D13: track 54.3 -> 0.00 mm, vias 2 -> 0
- net /A0: track 0.00 -> 48.0 mm
- net +12V: track 41.6 -> 50.6 mm
- net /5V: track 44.8 -> 41.4 mm
- net Net-(D1-Pad2): track 53.4 -> 55.9 mm
Other:
- board outline added: 63.5 x 53.3 mm

Commit message: -Add gerber files
Parts:
- added C3: C, FootprintGamelGe2_v6:C_Rect_L7.0mm_W2.5mm_P5.00mm, F.Cu at (217.2, 87.0)
Routing:
- net GND: track 154.9 -> 158.3 mm
- net /A0: track 48.0 -> 49.6 mm
- added copper zone on B.Cu, net GND
- added copper zone on F.Cu, net GND
Other:
- board text added: "LP pro MECSE Antoine BROUZES 2022-2023"
Changed lines of the file:
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@@
     (pad_to_mask_clearance 0)
     (pcbplotparams
-      (layerselection 0x00010fc_ffffffff)
+      (layerselection 0x0001c00_ffffffff)
       (disableapertmacros false)
-      (usegerberextensions false)
+      (usegerberextensions true)
       (usegerberattributes true)
       (usegerberadvancedattributes true)
-      (creategerberjobfile true)
+      (creategerberjobfile false)
       (svguseinch false)
       (svgprecision 6)
@@
       (outputformat 1)
       (mirror false)
-      (drillshape 1)
+      (drillshape 0)
       (scaleselection 1)
-      (outputdirectory "")
+      (outputdirectory "../Gerber/")
     )
   )
@@
     )
   )
+  (footprint "FootprintGamelGe2_v6:C_Rect_L7.0mm_W2.5mm_P5.00mm" (layer "F.Cu")
+    (at 217.17 86.995)
+    (descr "C, Rect series, Radial, pin pitch=5.00mm, , length*width=7*2.5mm^2, Capacitor")
+    (tags "C Rect series Radial pin pitch 5.00mm  length 7mm width 2.5mm Capacitor")
+    (property "Sheetfile" "Système_PCB.kicad_sch")
+    (property "Sheetname" "")
+    (attr through_hole)
+    (fp_text reference "C3" (at 2.5 -2.5) (layer "F.SilkS")
+      (effects (font (size 1 1) (thickness 0.15)))
+    )
+    (fp_text value "C" (at 2.5 2.5) (layer "F.Fab")
+      (effects (font (size 1 1) (thickness 0.15)))
+    )
+    (fp_text user "${REFERENCE}" (at 2.5 0) (layer "F.Fab")
+      (effects (font (size 1 1) (thickness 0.15)))
+    )
+    (fp_line (start -1.12 -1.37) (end -1.12 1.37) (layer "F.SilkS") (width 0.12))
+    (fp_line (start -1.12 -1.37) (end 6.12 -1.37) (layer "F.SilkS") (width 0.12))
+    (fp_line (start -1.12 1.37) (end 6.12 1.37) (layer "F.SilkS") (width 0.12))
+    (fp_line (start 6.12 -1.37) (end 6.12 1.37) (layer "F.SilkS") (width 0.12))
+    (fp_line (start -1.25 1.5) (end 6.25 1.5) (layer "F.CrtYd") (width 0.05))
+    (fp_line (start 6.25 1.5) (end 6.25 -1.5) (layer "F.CrtYd") (width 0.05))
+    (fp_line (start 6.25 -1.5) (end -1.25 -1.5) (layer "F.CrtYd") (width 0.05))
+    (fp_line (start -1.25 -1.5) (end -1.25 1.5) (layer "F.CrtYd") (width 0.05))
+    (fp_line (start -1 1.25) (end 6 1.25) (layer "F.Fab") (width 0.1))
+    (fp_line (start -1 -1.25) (end -1 1.25) (layer "F.Fab") (width 0.1))
+    (fp_line (start 6 -1.25) (end -1 -1.25) (layer "F.Fab") (width 0.1))
+    (fp_line (start 6 1.25) (end 6 -1.25) (layer "F.Fab") (width 0.1))
+    (pad "1" thru_hole circle (at 0 0) (size 1.8 1.8) (drill 0.8) (layers *.Cu *.Mask)
+      (net 1 "+12V") (pintype "passive"))
+    (pad "2" thru_hole circle (at 5 0) (size 1.8 1.8) (drill 0.8) (layers *.Cu *.Mask)
+      (net 6 "GND") (pintype "passive"))
+    (model "${KIPRJMOD}/LibGamelGe2_v6/3D/C_Rect_L7.0mm_W2.5mm_P5.00mm.STEP"
+      (offset (xyz 2.5 0.1 0))
+      (scale (xyz 1 1 1))
+      (rotate (xyz 0 0 0))
+    )
+  )
   (footprint "FootprintGamelGe2_v6:OmnimateSL-5,08_1x02_P5.08mm_Vertical" (layer "F.Cu")
     (at 203.2 66.04 -90)
@@
   (gr_line (start 259.08 52.07) (end 259.08 105.41) (layer "Edge.Cuts") (width 0.1))
   (gr_line (start 195.58 52.07) (end 259.08 52.07) (layer "Edge.Cuts") (width 0.1))
+  (gr_text "LP pro MECSE\nAntoine BROUZES\n2022-2023" (at 205.105 100.33) (layer "B.Cu")
+    (effects (font (size 1.2 1.2) (thickness 0.3)) (justify mirror))
+  )
   (gr_text "+" (at 200.66 92.71 270) (layer "Eco1.User")
     (effects (font (size 1.5 1.5) (thickness 0.3)))
@@
   (segment (start 222.25 83.82) (end 224.79 83.82) (width 1.25) (layer "B.Cu") (net 2))
   (segment (start 224.79 83.82) (end 227.33 81.28) (width 1.25) (layer "B.Cu") (net 2))
-  (segment (start 251.445 71.095) (end 251.435 71.095) (width 0.5) (layer "F.Cu") (net 6))
   (segment (start 238.125 88.9) (end 230.505 96.52) (width 0.5) (layer "F.Cu") (net 6))
   (segment (start 240.665 88.9) (end 238.125 88.9) (width 0.5) (layer "F.Cu") (net 6))
@@
   (segment (start 217.17 64.77) (end 217.17 61.595) (width 0.5) (layer "B.Cu") (net 6))
   (segment (start 204.47 64.77) (end 203.2 66.04) (width 0.5) (layer "B.Cu") (net 6))
+  (segment (start 237.49 76.292323) (end 224.836162 88.946162) (width 0.5) (layer "B.Cu") (net 6))
   (segment (start 217.17 64.77) (end 204.47 64.77) (width 0.5) (layer "B.Cu") (net 6))
   (segment (start 242.57 62.23) (end 237.15 62.23) (width 0.5) (layer "B.Cu") (net 6))
   (segment (start 240.665 88.9) (end 237.49 85.725) (width 0.5) (layer "B.Cu") (net 6))
   (segment (start 251.445 71.095) (end 251.435 71.095) (width 0.5) (layer "B.Cu") (net 6))
-  (segment (start 237.49 76.292323) (end 217.17 96.612323) (width 0.5) (layer "B.Cu") (net 6))
+  (segment (start 222.17 86.995) (end 224.121162 88.946162) (width 0.5) (layer "B.Cu") (net 6))
   (segment (start 245.11 64.77) (end 237.49 72.39) (width 0.5) (layer "B.Cu") (net 6))
+  (segment (start 224.121162 88.946162) (end 224.836162 88.946162) (width 0.5) (layer "B.Cu") (net 6))
   (segment (start 237.49 76.2) (end 237.49 76.292323) (width 0.5) (layer "B.Cu") (net 6))
   (segment (start 251.435 71.095) (end 242.57 62.23) (width 0.5) (layer "B.Cu") (net 6))
+  (segment (start 224.836162 88.946162) (end 217.17 96.612323) (width 0.5) (layer "B.Cu") (net 6))
   (segment (start 237.49 72.39) (end 237.49 76.2) (width 0.5) (layer "B.Cu") (net 6))
   (segment (start 217.17 66.04) (end 219.075 67.945) (width 0.5) (layer "B.Cu") (net 6))
@@
   (segment (start 251.445 78.715) (end 251.445 80.025) (width 0.5) (layer "B.Cu") (net 9))
   (segment (start 242.61 81.32) (end 242.57 81.28) (width 0.5) (layer "B.Cu") (net 9))
-  (segment (start 248.895 76.175) (end 243.84 71.12) (width 0.5) (layer "F.Cu") (net 10))
-  (segment (start 238.76 100.33) (end 238.125 100.965) (width 0.5) (layer "F.Cu") (net 10))
-  (segment (start 252.645 76.175) (end 254 77.53) (width 0.5) (layer "F.Cu") (net 10))
+  (segment (start 242.57 73.025) (end 248.92 79.375) (width 0.5) (layer "F.Cu") (net 10))
+  (segment (start 248.92 79.375) (end 248.92 90.17) (width 0.5) (layer "F.Cu") (net 10))
+  (segment (start 248.92 90.17) (end 238.125 100.965) (width 0.5) (layer "F.Cu") (net 10))
+  (segment (start 242.57 71.12) (end 242.57 73.025) (width 0.5) (layer "F.Cu") (net 10))
   (segment (start 238.125 100.965) (end 238.125 102.616) (width 0.5) (layer "F.Cu") (net 10))
-  (segment (start 243.84 71.12) (end 242.57 71.12) (width 0.5) (layer "F.Cu") (net 10))
-  (segment (start 254 88.9) (end 242.57 100.33) (width 0.5) (layer "F.Cu") (net 10))
-  (segment (start 242.57 100.33) (end 238.76 100.33) (width 0.5) (layer "F.Cu") (net 10))
-  (segment (start 251.445 76.175) (end 252.645 76.175) (width 0.5) (layer "F.Cu") (net 10))
-  (segment (start 251.445 76.175) (end 248.895 76.175) (width 0.5) (layer "F.Cu") (net 10))
-  (segment (start 254 77.53) (end 254 88.9) (width 0.5) (layer "F.Cu") (net 10))
+  (segment (start 250.8 76.175) (end 245.745 71.12) (width 0.5) (layer "B.Cu") (net 10))
+  (segment (start 245.745 71.12) (end 242.57 71.12) (width 0.5) (layer "B.Cu") (net 10))
+  (segment (start 251.445 76.175) (end 250.8 76.175) (width 0.5) (layer "B.Cu") (net 10))
   (segment (start 237.15 59.69) (end 245.11 59.69) (width 0.5) (layer "F.Cu") (net 19))
   (segment (start 245.11 59.69) (end 248.285 56.515) (width 0.5) (layer "F.Cu") (net 19))
@@
   (segment (start 248.285 56.515) (end 248.285 54.61) (width 0.5) (layer "F.Cu") (net 19))
   (segment (start 237.15 59.69) (end 231.14 59.69) (width 0.5) (layer "F.Cu") (net 19))
+  (zone (net 6) (net_name "GND") (layers F&B.Cu) (hatch edge 0.508)
+    (connect_pads (clearance 0.508))
+    (min_thickness 0.254) (filled_areas_thickness no)
+    (fill yes (thermal_gap 0.508) (thermal_bridge_width 0.508))
+    (polygon
+      (pts
+        (xy 259.08 105.41)
+        (xy 195.58 105.41)
+        (xy 195.58 52.07)
+        (xy 259.08 52.07)
+      )
+    )
+  )
 )

Commit message: -add PWM
Parts:
- C1, C3: value C -> 20n
- C2: value Cp -> 100µ; footprint FootprintGamelGe2_v6:CP_Radial_D10.0mm_P5.00mm -> FootprintGamelGe2_v6:CP_Radial_D5.0mm_P2.50mm
- R1: value R -> 1k
- R2: value R -> 4.7k
Routing:
- net GND: track 158.3 -> 147.5 mm

Commit message: --Add DHT library
Connections:
- Q1 pad 2: GND -> Net-(D1-Pad2)
- Q1 pad 3: Net-(D1-Pad2) -> GND
Routing:
- net GND: track 147.5 -> 113.2 mm, vias 2 -> 0
Changed lines of the file:
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@@
       (net 19 "/D1") (pinfunction "G") (pintype "input"))
     (pad "2" thru_hole oval (at 2.54 0 270) (size 2 2.5) (drill 1) (layers *.Cu *.Mask)
-      (net 6 "GND") (pinfunction "D") (pintype "passive"))
+      (net 2 "Net-(D1-Pad2)") (pinfunction "D") (pintype "passive"))
     (pad "3" thru_hole oval (at 5.08 0 270) (size 2 2.5) (drill 1) (layers *.Cu *.Mask)
-      (net 2 "Net-(D1-Pad2)") (pinfunction "S") (pintype "passive"))
+      (net 6 "GND") (pinfunction "S") (pintype "passive"))
     (model "${KIPRJMOD}/LibGamelGe2_v6/3D/TO220_horizontal.STEP"
       (offset (xyz 2.54 4.3 0))
@@
   (segment (start 215.9 69.85) (end 217.17 71.12) (width 1.25) (layer "B.Cu") (net 1))
   (segment (start 222.25 83.82) (end 215.9 83.82) (width 1.25) (layer "F.Cu") (net 2))
+  (segment (start 235.15 62.23) (end 227.33 70.05) (width 1.25) (layer "F.Cu") (net 2))
+  (segment (start 237.15 62.23) (end 235.15 62.23) (width 1.25) (layer "F.Cu") (net 2))
   (segment (start 215.9 83.82) (end 210.82 78.74) (width 1.25) (layer "F.Cu") (net 2))
   (segment (start 210.82 78.74) (end 205.74 78.74) (width 1.25) (layer "F.Cu") (net 2))
+  (segment (start 227.33 70.05) (end 227.33 72.39) (width 1.25) (layer "F.Cu") (net 2))
   (via (at 222.25 83.82) (size 2) (drill 0.7) (layers "F.Cu" "B.Cu") (net 2))
   (via (at 205.74 78.74) (size 2) (drill 0.7) (layers "F.Cu" "B.Cu") (net 2))
   (segment (start 204.47 78.74) (end 205.74 78.74) (width 1.25) (layer "B.Cu") (net 2))
   (segment (start 203.2 80.01) (end 204.47 78.74) (width 1.25) (layer "B.Cu") (net 2))
-  (segment (start 233.68 72.39) (end 227.33 72.39) (width 1.25) (layer "B.Cu") (net 2))
-  (segment (start 237.15 68.92) (end 233.68 72.39) (width 1.25) (layer "B.Cu") (net 2))
   (segment (start 203.2 83.82) (end 203.2 80.01) (width 1.25) (layer "B.Cu") (net 2))
   (segment (start 227.33 81.28) (end 227.33 72.39) (width 1.25) (layer "B.Cu") (net 2))
-  (segment (start 237.15 64.77) (end 237.15 68.92) (width 1.25) (layer "B.Cu") (net 2))
   (segment (start 222.25 83.82) (end 224.79 83.82) (width 1.25) (layer "B.Cu") (net 2))
   (segment (start 224.79 83.82) (end 227.33 81.28) (width 1.25) (layer "B.Cu") (net 2))
@@
   (segment (start 230.505 96.52) (end 230.505 102.616) (width 0.5) (layer "F.Cu") (net 6))
   (segment (start 215.9 60.325) (end 213.745 58.17) (width 0.5) (layer "F.Cu") (net 6))
-  (via (at 240.665 88.9) (size 2) (drill 0.7) (layers "F.Cu" "B.Cu") (net 6))
-  (via (at 215.9 60.325) (size 2) (drill 0.7) (layers "F.Cu" "B.Cu") (net 6))
-  (segment (start 241.3 88.9) (end 240.665 88.9) (width 0.5) (layer "B.Cu") (net 6))
-  (segment (start 228.6 67.945) (end 234.315 62.23) (width 0.5) (layer "B.Cu") (net 6))
   (segment (start 217.17 64.77) (end 217.17 61.595) (width 0.5) (layer "B.Cu") (net 6))
   (segment (start 204.47 64.77) (end 203.2 66.04) (width 0.5) (layer "B.Cu") (net 6))
   (segment (start 237.49 76.292323) (end 224.836162 88.946162) (width 0.5) (layer "B.Cu") (net 6))
   (segment (start 217.17 64.77) (end 204.47 64.77) (width 0.5) (layer "B.Cu") (net 6))
-  (segment (start 242.57 62.23) (end 237.15 62.23) (width 0.5) (layer "B.Cu") (net 6))
   (segment (start 240.665 88.9) (end 237.49 85.725) (width 0.5) (layer "B.Cu") (net 6))
   (segment (start 251.445 71.095) (end 251.435 71.095) (width 0.5) (layer "B.Cu") (net 6))
   (segment (start 222.17 86.995) (end 224.121162 88.946162) (width 0.5) (layer "B.Cu") (net 6))
-  (segment (start 245.11 64.77) (end 237.49 72.39) (width 0.5) (layer "B.Cu") (net 6))
   (segment (start 224.121162 88.946162) (end 224.836162 88.946162) (width 0.5) (layer "B.Cu") (net 6))
   (segment (start 237.49 76.2) (end 237.49 76.292323) (width 0.5) (layer "B.Cu") (net 6))
-  (segment (start 251.435 71.095) (end 242.57 62.23) (width 0.5) (layer "B.Cu") (net 6))
+  (segment (start 237.15 72.05) (end 237.15 64.77) (width 0.5) (layer "B.Cu") (net 6))
+  (segment (start 237.49 72.39) (end 237.15 72.05) (width 0.5) (layer "B.Cu") (net 6))
   (segment (start 237.49 72.39) (end 237.49 76.2) (width 0.5) (layer "B.Cu") (net 6))
   (segment (start 217.17 66.04) (end 219.075 67.945) (width 0.5) (layer "B.Cu") (net 6))
   (segment (start 217.17 64.77) (end 217.17 66.04) (width 0.5) (layer "B.Cu") (net 6))
   (segment (start 237.49 85.725) (end 237.49 76.2) (width 0.5) (layer "B.Cu") (net 6))
-  (segment (start 234.315 62.23) (end 237.15 62.23) (width 0.5) (layer "B.Cu") (net 6))
-  (segment (start 217.17 61.595) (end 215.9 60.325) (width 0.5) (layer "B.Cu") (net 6))
   (segment (start 243.88 86.32) (end 241.3 88.9) (width 0.5) (layer "B.Cu") (net 6))
   (segment (start 219.075 67.945) (end 228.6 67.945) (width 0.5) (layer "B.Cu") (net 6))

Commit message: Add comment
Routing:
- net GND: track 113.2 -> 101.5 mm, vias 0 -> 2
Changed lines of the file:
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@@
   (segment (start 230.505 96.52) (end 230.505 102.616) (width 0.5) (layer "F.Cu") (net 6))
   (segment (start 215.9 60.325) (end 213.745 58.17) (width 0.5) (layer "F.Cu") (net 6))
+  (via (at 215.9 60.325) (size 2) (drill 0.7) (layers "F.Cu" "B.Cu") (net 6))
+  (via (at 241.3 88.9) (size 2) (drill 0.7) (layers "F.Cu" "B.Cu") (net 6))
   (segment (start 217.17 64.77) (end 217.17 61.595) (width 0.5) (layer "B.Cu") (net 6))
   (segment (start 204.47 64.77) (end 203.2 66.04) (width 0.5) (layer "B.Cu") (net 6))
@@
   (segment (start 237.49 72.39) (end 237.15 72.05) (width 0.5) (layer "B.Cu") (net 6))
   (segment (start 237.49 72.39) (end 237.49 76.2) (width 0.5) (layer "B.Cu") (net 6))
-  (segment (start 217.17 66.04) (end 219.075 67.945) (width 0.5) (layer "B.Cu") (net 6))
-  (segment (start 217.17 64.77) (end 217.17 66.04) (width 0.5) (layer "B.Cu") (net 6))
+  (segment (start 217.17 61.595) (end 215.9 60.325) (width 0.5) (layer "B.Cu") (net 6))
   (segment (start 237.49 85.725) (end 237.49 76.2) (width 0.5) (layer "B.Cu") (net 6))
   (segment (start 243.88 86.32) (end 241.3 88.9) (width 0.5) (layer "B.Cu") (net 6))
-  (segment (start 219.075 67.945) (end 228.6 67.945) (width 0.5) (layer "B.Cu") (net 6))
   (segment (start 246.38 86.32) (end 243.88 86.32) (width 0.5) (layer "B.Cu") (net 6))
   (segment (start 238.76 81.28) (end 225.425 94.615) (width 0.5) (layer "F.Cu") (net 9))
